File: child_1.kicad_sch (KiCad schematic)
At the start: 5 parts

Commit message: test dnp
Parts:
- R10: now fitted
Changed lines of the file:
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@@
 		(on_board yes)
 		(in_pos_files yes)
-		(dnp yes)
+		(dnp no)
 		(fields_autoplaced yes)
 		(property "Reference" "R10"

Commit message: test longer bom
Parts:
- added U1: STM32WBA55HEFx, Package_CSP:ST_WLCSP-41_2.98x2.76mm_Layout13x7_P0.4mm_Stagger, symbol MCU_ST_STM32WB:STM32WBA55HEFx
- R8: now not fitted
Connections:
- new net: U1.A10 (VDD), U1.A12 (VSSSMPS), U1.A6 (VDDRF), U1.A8 (OSC_IN), U1.B11 (VDD11), U1.B13 (VDDSMPS), U1.B5 (VDDANA), U1.B7 (OSC_OUT), U1.B9 (VSS), U1.C10 (PB12), U1.C12 (VLXSMPS), U1.C2 (RF), U1.C4 (VDDHPA), U1.C6 (VDDRFPA), U1.C8 (PH3), U1.D1 (VSSRF), U1.D11 (PA7), U1.D13 (VSSA), U1.D3 (VSSRF), U1.D5 (VSSRF), U1.D7 (PA8), U1.D9 (PA6), U1.E10 (PA1), U1.E12 (VDDA), U1.E2 (NRST), U1.E4 (PB15), U1.E6 (PA12), U1.E8 (PA13), U1.F1 (PA14), U1.F11 (PA2), U1.F13 (PA5), U1.F3 (PA15), U1.F5 (PB4), U1.F7 (PC15), U1.F9 (PB9), U1.G10 (PB8), U1.G12 (PA0), U1.G2 (PB3), U1.G4 (VDD), U1.G6 (VSS), U1.G8 (PC14)
