File: ktest.kicad_sch (KiCad schematic)
At the start: 13 parts, among them J1 Conn_01x03_Pin

Commit message: testing hierarchical sheets
Parts:
- added R6, R7: 10k, Resistor_SMD:R_01005_0402Metric, symbol Device:R
- C2, R5: now not fitted
Connections:
- net at C2.1, J1.3 (Pin_3), R2.1: now also R7.1
- net at C1.1, C2.2, R1.1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: now also R6.1, R7.2
- net child_1/a: now reaches R4.2, R5.2
- net child_1/n: now reaches C3.1, D1.1 (K), J1.1 (Pin_1), R3.1
- net at C1.2, J1.2 (Pin_2), R1.2: now also R6.2
Other:
- added sheet child_1 (child_1.kicad_sch)

Commit message: test dnp
Parts:
- R4: now not fitted
Changed lines of the file:
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@@
 		(on_board yes)
 		(in_pos_files yes)
-		(dnp no)
+		(dnp yes)
 		(fields_autoplaced yes)
 		(property "Reference" "R4"

Commit message: test longer bom
Parts:
- added C10: 6p, Capacitor_SMD:C_0603_1608Metric_Pad1.08x0.95mm_HandSolder, symbol Device:C
- added C11: 9p, Capacitor_SMD:C_0603_1608Metric_Pad1.08x0.95mm_HandSolder, symbol Device:C
- added C12: 5p, Capacitor_SMD:C_0603_1608Metric_Pad1.08x0.95mm_HandSolder, symbol Device:C
- added C13: 8p, Capacitor_SMD:C_0603_1608Metric_Pad1.08x0.95mm_HandSolder, symbol Device:C
- added C14: 10p, Capacitor_SMD:C_0603_1608Metric_Pad1.08x0.95mm_HandSolder, symbol Device:C
- added C15: 11p, Capacitor_SMD:C_0603_1608Metric_Pad1.08x0.95mm_HandSolder, symbol Device:C
- added C16: 12p, Capacitor_SMD:C_0603_1608Metric_Pad1.08x0.95mm_HandSolder, symbol Device:C
- added C17: 16p, Capacitor_SMD:C_0603_1608Metric_Pad1.08x0.95mm_HandSolder, symbol Device:C
- added C18: 15p, Capacitor_SMD:C_0603_1608Metric_Pad1.08x0.95mm_HandSolder, symbol Device:C
- added C19: 14p, Capacitor_SMD:C_0603_1608Metric_Pad1.08x0.95mm_HandSolder, symbol Device:C
- added C20: 13p, Capacitor_SMD:C_0603_1608Metric_Pad1.08x0.95mm_HandSolder, symbol Device:C
- added C5: 1p, Capacitor_SMD:C_0603_1608Metric_Pad1.08x0.95mm_HandSolder, symbol Device:C
- added C6: 2p, Capacitor_SMD:C_0603_1608Metric_Pad1.08x0.95mm_HandSolder, symbol Device:C
- added C7: 3p, Capacitor_SMD:C_0603_1608Metric_Pad1.08x0.95mm_HandSolder, symbol Device:C
- added C8: 4p, Capacitor_SMD:C_0603_1608Metric_Pad1.08x0.95mm_HandSolder, symbol Device:C
- added C9: 7p, Capacitor_SMD:C_0603_1608Metric_Pad1.08x0.95mm_HandSolder, symbol Device:C
- added R11: 1k, Resistor_SMD:R_0805_2012Metric_Pad1.20x1.40mm_HandSolder, symbol Device:R
- added R12: 2k2, Resistor_SMD:R_0805_2012Metric_Pad1.20x1.40mm_HandSolder, symbol Device:R
- added R13: 3k3, Resistor_SMD:R_0805_2012Metric_Pad1.20x1.40mm_HandSolder, symbol Device:R
- added R14: 4k7, Resistor_SMD:R_0805_2012Metric_Pad1.20x1.40mm_HandSolder, symbol Device:R
- added R15: 5k1, Resistor_SMD:R_0805_2012Metric_Pad1.20x1.40mm_HandSolder, symbol Device:R
- added R16: 5k6, Resistor_SMD:R_0805_2012Metric_Pad1.20x1.40mm_HandSolder, symbol Device:R
- added R17: 6k8, Resistor_SMD:R_0805_2012Metric_Pad1.20x1.40mm_HandSolder, symbol Device:R
- added R18: 7k5, Resistor_SMD:R_0805_2012Metric_Pad1.20x1.40mm_HandSolder, symbol Device:R
- added R19: 9k1, Resistor_SMD:R_0805_2012Metric_Pad1.20x1.40mm_HandSolder, symbol Device:R
Connections:
- net child_1/a: now also R11.1, R12.1, R13.1
- new net: C10.2, C11.2, C12.2, C13.1, C14.1, C15.1, C16.1, C17.2, C18.2, C19.2, C20.2, C5.1, C6.1, C7.1, C8.1, C9.2
- new net: C10.1, C11.1, C12.1, C13.2, C14.2, C15.2, C16.2, C17.1, C18.1, C19.1, C20.1, C5.2, C6.2, C7.2, C8.2, C9.1
- new net: R13.2, R16.1
- new net: R16.2, R19.1
- new net: R12.2, R15.1
- new net: R15.2, R18.1
- new net: R14.2, R17.1
- new net: R17.2, R18.2, R19.2
- new net: R11.2, R14.1

Commit message: new wks template
Other:
- title: Kibot test -> 1 kV strobe
Changed lines of the file:
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@@
 	(paper "A4")
 	(title_block
-		(title "Kibot test")
-		(date "2026-09-30")
+		(title "1 kV strobe")
+		(date "2026/09/30")
 		(rev "0.0.1")
 		(company "Example company")
-		(comment 1 "comm1")
-		(comment 2 "comm2")
-		(comment 3 "comm3")
-		(comment 4 "comm4")
-		(comment 5 "comm5")
+		(comment 1 "This is a comment 1 field - potentially not used")
+		(comment 2 "This is a comment 2 field - potentially not used")
+		(comment 3 "This is a comment 3 field - potentially not used")
+		(comment 4 "This is a comment 4 field - potentially not used")
+		(comment 5 "This is a comment 5 field - potentially not used")
 	)
 	(junction

Commit message: testing erc bypass
Parts:
- added U2: ATmega8-16P, Package_DIP:DIP-28_W7.62mm, symbol MCU_Microchip_ATmega:ATmega8-16P
Changed lines of the file:
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@@
+	)
+	(symbol
+		(lib_id "MCU_Microchip_ATmega:ATmega8-16P")
+		(at 41.91 140.97 0)
+		(unit 1)
+		(body_style 1)
+		(exclude_from_sim no)
+		(in_bom yes)
+		(on_board yes)
+		(in_pos_files yes)
+		(dnp no)
+		(fields_autoplaced yes)
+		(property "Reference" "U2"
+			(at 46.5933 102.87 0)
+			(show_name no)
+			(do_not_autoplace no)
+			(effects
+				(font
+					(size 1.27 1.27)
+				)
+				(justify left)
+			)
+		)
+		(property "Value" "ATmega8-16P"
+			(at 46.5933 105.41 0)
+			(show_name no)
+			(do_not_autoplace no)
+			(effects
+				(font
+					(size 1.27 1.27)
+				)
+				(justify left)
+			)
+		)
+		(property "Footprint" "Package_DIP:DIP-28_W7.62mm"
+			(at 41.91 140.97 0)
+			(hide yes)
+			(show_name no)
+			(do_not_autoplace no)
+			(effects
+				(font
+					(size 1.27 1.27)
+					(italic yes)
+				)
+			)
+		)
+		(property "Datasheet" "http://ww1.microchip.com/downloads/en/DeviceDoc/atmel-2486-8-bit-avr-microcontroller-atmega8_l_datasheet.pdf"
+			(at 41.91 140.97 0)
+			(hide yes)
+			(show_name no)
+			(do_not_autoplace no)
+			(effects
+				(font
+					(size 1.27 1.27)
+				)
+			)
+		)
+		(property "Description" "16MHz, 8kB Flash, 1kB SRAM, 512B EEPROM, DIP-28"
+			(at 41.91 140.97 0)
+			(hide yes)
+			(show_name no)
+			(do_not_autoplace no)
+			(effects
+				(font
+					(size 1.27 1.27)
+				)
+			)
+		)
+		(pin "13"
+		)
+		(pin "15"
+		)
+		(pin "2"
+		)
+		(pin "4"
+		)
+		(pin "12"
+		)
+		(pin "14"
+		)
+		(pin "22"
+		)
+		(pin "23"
+		)
+		(pin "16"
+		)
+		(pin "18"
+		)
+		(pin "9"
+		)
+		(pin "5"
+		)
+		(pin "19"
+		)
+		(pin "20"
+		)
+		(pin "10"
+		)
+		(pin "8"
+		)
+		(pin "6"
+		)
+		(pin "11"
+		)
+		(pin "21"
+		)
+		(pin "7"
+		)
+		(pin "27"
+		)
+		(pin "28"
+		)
+		(pin "25"
+		)
+		(pin "26"
+		)
+		(pin "3"
+		)
+		(pin "17"
+		)
+		(pin "1"
+		)
+		(pin "24"
+		)
+		(instances
+			(project "ktest"
+				(path "/f14ff7c3-fe34-4697-84b8-3cc06a5a3565"
+					(reference "U2")
+					(unit 1)
+				)
+			)
+		)
 	)
 	(symbol

Commit message: testing both erc drc overlay
Connections:
- net at U2.14 (PB0): now also U2.15 (PB1), U2.16 (PB2), U2.17 (PB3), U2.18 (PB4), U2.19 (PB5), U2.2 (PD0), U2.23 (PC0), U2.24 (PC1), U2.25 (PC2), U2.26 (PC3), U2.27 (PC4), U2.28 (PC5), U2.3 (PD1), U2.4 (PD2)
Changed lines of the file:
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@@
+	)
+	(junction
+		(at 57.15 138.43)
+		(diameter 0)
+		(color 0 0 0 0)
 	)
 	(junction
@@
 	)
 	(junction
+		(at 57.15 130.81)
+		(diameter 0)
+		(color 0 0 0 0)
+	)
+	(junction
 		(at 241.3 107.95)
 		(diameter 0)
@@
 	)
 	(junction
+		(at 57.15 143.51)
+		(diameter 0)
+		(color 0 0 0 0)
+	)
+	(junction
 		(at 228.6 118.11)
 		(diameter 0)
@@
 	)
 	(junction
+		(at 57.15 120.65)
+		(diameter 0)
+		(color 0 0 0 0)
+	)
+	(junction
 		(at 228.6 86.36)
 		(diameter 0)
@@
 	)
 	(junction
+		(at 57.15 148.59)
+		(diameter 0)
+		(color 0 0 0 0)
+	)
+	(junction
 		(at 266.7 97.79)
 		(diameter 0)
@@
 	)
 	(junction
+		(at 57.15 151.13)
+		(diameter 0)
+		(color 0 0 0 0)
+	)
+	(junction
+		(at 57.15 123.19)
+		(diameter 0)
+		(color 0 0 0 0)
+	)
+	(junction
+		(at 57.15 140.97)
+		(diameter 0)
+		(color 0 0 0 0)
+	)
+	(junction
 		(at 266.7 118.11)
 		(diameter 0)
@@
 	)
 	(junction
+		(at 57.15 133.35)
+		(diameter 0)
+		(color 0 0 0 0)
+	)
+	(junction
 		(at 142.24 77.47)
 		(diameter 0)
@@
 	)
 	(junction
+		(at 57.15 125.73)
+		(diameter 0)
+		(color 0 0 0 0)
+	)
+	(junction
+		(at 57.15 118.11)
+		(diameter 0)
+		(color 0 0 0 0)
+	)
+	(junction
+		(at 57.15 135.89)
+		(diameter 0)
+		(color 0 0 0 0)
+	)
+	(junction
+		(at 57.15 115.57)
+		(diameter 0)
+		(color 0 0 0 0)
+	)
+	(junction
 		(at 241.3 97.79)
 		(diameter 0)
@@
 	(wire
 		(pts
+			(xy 57.15 133.35) (xy 57.15 135.89)
+		)
+		(stroke
+			(width 0)
+			(type default)
+		)
+	)
+	(wire
+		(pts
 			(xy 254 86.36) (xy 254 88.9)
 		)
@@
 	(wire
 		(pts
+			(xy 57.15 143.51) (xy 57.15 148.59)
+		)
+		(stroke
+			(width 0)
+			(type default)
+		)
+	)
+	(wire
+		(pts
 			(xy 66.04 105.41) (xy 66.04 111.76)
 		)
@@
 	(wire
 		(pts
+			(xy 57.15 135.89) (xy 57.15 138.43)
+		)
+		(stroke
+			(width 0)
+			(type default)
+		)
+	)
+	(wire
+		(pts
 			(xy 105.41 82.55) (xy 110.49 82.55)
 		)
@@
 	(wire
 		(pts
+			(xy 57.15 123.19) (xy 57.15 125.73)
+		)
+		(stroke
+			(width 0)
+			(type default)
+		)
+	)
+	(wire
+		(pts
 			(xy 266.7 128.27) (xy 254 128.27)
 		)
@@
 	(wire
 		(pts
+			(xy 57.15 151.13) (xy 57.15 153.67)
+		)
+		(stroke
+			(width 0)
+			(type default)
+		)
+	)
+	(wire
+		(pts
 			(xy 228.6 97.79) (xy 241.3 97.79)
 		)
@@
 	(wire
 		(pts
+			(xy 57.15 125.73) (xy 57.15 130.81)
+		)
+		(stroke
+			(width 0)
+			(type default)
+		)
+	)
+	(wire
+		(pts
 			(xy 241.3 99.06) (xy 241.3 97.79)
 		)
@@
 	(wire
 		(pts
+			(xy 57.15 120.65) (xy 57.15 123.19)
+		)
+		(stroke
+			(width 0)
+			(type default)
+		)
+	)
+	(wire
+		(pts
 			(xy 207.01 50.8) (xy 207.01 49.53)
 		)
@@
 	(wire
 		(pts
+			(xy 57.15 148.59) (xy 57.15 151.13)
+		)
+		(stroke
+			(width 0)
+			(type default)
+		)
+	)
+	(wire
+		(pts
 			(xy 90.17 105.41) (xy 90.17 111.76)
 		)
@@
 	(wire
 		(pts
+			(xy 57.15 118.11) (xy 57.15 120.65)
+		)
+		(stroke
+			(width 0)
+			(type default)
+		)
+	)
+	(wire
+		(pts
 			(xy 254 107.95) (xy 266.7 107.95)
 		)
@@
 	(wire
 		(pts
+			(xy 57.15 138.43) (xy 57.15 140.97)
+		)
+		(stroke
+			(width 0)
+			(type default)
+		)
+	)
+	(wire
+		(pts
 			(xy 156.21 104.14) (xy 156.21 110.49)
 		)
@@
 	(wire
 		(pts
+			(xy 57.15 113.03) (xy 57.15 115.57)
+		)
+		(stroke
+			(width 0)
+			(type default)
+		)
+	)
+	(wire
+		(pts
 			(xy 207.01 59.69) (xy 207.01 58.42)
 		)
@@
 	(wire
 		(pts
+			(xy 57.15 130.81) (xy 57.15 133.35)
+		)
+		(stroke
+			(width 0)
+			(type default)
+		)
+	)
+	(wire
+		(pts
 			(xy 66.04 90.17) (xy 76.2 90.17)
 		)
@@
 		)
 		(stroke
+			(width 0)
+			(type default)
+		)
+	)
+	(wire
+		(pts
+			(xy 57.15 140.97) (xy 57.15 143.51)
+		)
+		(stroke
+			(width 0)
+			(type default)
+		)
+	)
+	(wire
+		(pts
+			(xy 57.15 115.57) (xy 57.15 118.11)
+		)
+		(stroke

Commit message: testing drc bypass only
Connections:
- now unconnected: U2.14 (PB0), U2.15 (PB1), U2.16 (PB2), U2.17 (PB3), U2.18 (PB4), U2.19 (PB5), U2.2 (PD0), U2.23 (PC0), U2.24 (PC1), U2.25 (PC2), U2.26 (PC3), U2.27 (PC4), U2.28 (PC5), U2.3 (PD1), U2.4 (PD2)
- no-connect marks 0 -> 28
Other:
- moved on the sheet: U2
Changed lines of the file:
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@@
-	)
-	(junction
-		(at 57.15 138.43)
-		(diameter 0)
-		(color 0 0 0 0)
 	)
 	(junction
@@
 	)
 	(junction
-		(at 57.15 130.81)
-		(diameter 0)
-		(color 0 0 0 0)
-	)
-	(junction
 		(at 241.3 107.95)
 		(diameter 0)
@@
 	)
 	(junction
-		(at 57.15 143.51)
-		(diameter 0)
-		(color 0 0 0 0)
-	)
-	(junction
 		(at 228.6 118.11)
 		(diameter 0)
@@
 	)
 	(junction
-		(at 57.15 120.65)
-		(diameter 0)
-		(color 0 0 0 0)
-	)
-	(junction
 		(at 228.6 86.36)
 		(diameter 0)
@@
 	)
 	(junction
-		(at 57.15 148.59)
-		(diameter 0)
-		(color 0 0 0 0)
-	)
-	(junction
 		(at 266.7 97.79)
 		(diameter 0)
@@
 	)
 	(junction
-		(at 57.15 151.13)
-		(diameter 0)
-		(color 0 0 0 0)
-	)
-	(junction
-		(at 57.15 123.19)
-		(diameter 0)
-		(color 0 0 0 0)
-	)
-	(junction
-		(at 57.15 140.97)
-		(diameter 0)
-		(color 0 0 0 0)
-	)
-	(junction
 		(at 266.7 118.11)
 		(diameter 0)
@@
 	)
 	(junction
-		(at 57.15 133.35)
-		(diameter 0)
-		(color 0 0 0 0)
-	)
-	(junction
 		(at 142.24 77.47)
 		(diameter 0)
@@
 	)
 	(junction
-		(at 57.15 125.73)
-		(diameter 0)
-		(color 0 0 0 0)
-	)
-	(junction
-		(at 57.15 118.11)
-		(diameter 0)
-		(color 0 0 0 0)
-	)
-	(junction
-		(at 57.15 135.89)
-		(diameter 0)
-		(color 0 0 0 0)
-	)
-	(junction
-		(at 57.15 115.57)
-		(diameter 0)
-		(color 0 0 0 0)
-	)
-	(junction
 		(at 241.3 97.79)
 		(diameter 0)
@@
 		(color 0 0 0 0)
 	)
+	(no_connect
+		(at 64.77 148.59)
+	)
+	(no_connect
+		(at 34.29 123.19)
+	)
+	(no_connect
+		(at 64.77 123.19)
+	)
+	(no_connect
+		(at 64.77 158.75)
+	)
+	(no_connect
+		(at 34.29 128.27)
+	)
+	(no_connect
+		(at 64.77 166.37)
+	)
+	(no_connect
+		(at 64.77 130.81)
+	)
+	(no_connect
+		(at 64.77 173.99)
+	)
+	(no_connect
+		(at 34.29 138.43)
+	)
+	(no_connect
+		(at 64.77 161.29)
+	)
+	(no_connect
+		(at 64.77 135.89)
+	)
+	(no_connect
+		(at 64.77 153.67)
+	)
+	(no_connect
+		(at 64.77 163.83)
+	)
+	(no_connect
+		(at 64.77 176.53)
+	)
+	(no_connect
+		(at 52.07 115.57)
+	)
+	(no_connect
+		(at 64.77 128.27)
+	)
+	(no_connect
+		(at 49.53 186.69)
+	)
+	(no_connect
+		(at 64.77 151.13)
+	)
+	(no_connect
+		(at 34.29 133.35)
+	)
+	(no_connect
+		(at 64.77 140.97)
+	)
+	(no_connect
+		(at 64.77 125.73)
+	)
+	(no_connect
+		(at 64.77 143.51)
+	)
+	(no_connect
+		(at 52.07 186.69)
+	)
+	(no_connect
+		(at 64.77 146.05)
+	)
+	(no_connect
+		(at 64.77 168.91)
+	)
+	(no_connect
+		(at 64.77 133.35)
+	)
+	(no_connect
+		(at 64.77 171.45)
+	)
+	(no_connect
+		(at 49.53 115.57)
+	)
 	(wire
 		(pts
@@
 	(wire
 		(pts
-			(xy 57.15 133.35) (xy 57.15 135.89)
-		)
-		(stroke
-			(width 0)
-			(type default)
-		)
-	)
-	(wire
-		(pts
 			(xy 254 86.36) (xy 254 88.9)
 		)
@@
 	(wire
 		(pts
-			(xy 57.15 143.51) (xy 57.15 148.59)
-		)
-		(stroke
-			(width 0)
-			(type default)
-		)
-	)
-	(wire
-		(pts
 			(xy 66.04 105.41) (xy 66.04 111.76)
 		)
@@
 	(wire
 		(pts
-			(xy 57.15 135.89) (xy 57.15 138.43)
-		)
-		(stroke
-			(width 0)
-			(type default)
-		)
-	)
-	(wire
-		(pts
 			(xy 105.41 82.55) (xy 110.49 82.55)
 		)
@@
 	(wire
 		(pts
-			(xy 57.15 123.19) (xy 57.15 125.73)
-		)
-		(stroke
-			(width 0)
-			(type default)
-		)
-	)
-	(wire
-		(pts
 			(xy 266.7 128.27) (xy 254 128.27)
 		)
@@
 	(wire
 		(pts
-			(xy 57.15 151.13) (xy 57.15 153.67)
-		)
-		(stroke
-			(width 0)
-			(type default)
-		)
-	)
-	(wire
-		(pts
 			(xy 228.6 97.79) (xy 241.3 97.79)
 		)
@@
 	(wire
 		(pts
-			(xy 57.15 125.73) (xy 57.15 130.81)
-		)
-		(stroke
-			(width 0)
-			(type default)
-		)
-	)
-	(wire
-		(pts
 			(xy 241.3 99.06) (xy 241.3 97.79)
 		)
@@
 	(wire
 		(pts
-			(xy 57.15 120.65) (xy 57.15 123.19)
-		)
-		(stroke
-			(width 0)
-			(type default)
-		)
-	)
-	(wire
-		(pts
 			(xy 207.01 50.8) (xy 207.01 49.53)
 		)
@@
 	(wire
 		(pts
-			(xy 57.15 148.59) (xy 57.15 151.13)
-		)
-		(stroke
-			(width 0)
-			(type default)
-		)
-	)
-	(wire
-		(pts
 			(xy 90.17 105.41) (xy 90.17 111.76)
 		)
@@
 	(wire
 		(pts
-			(xy 57.15 118.11) (xy 57.15 120.65)
-		)
-		(stroke
-			(width 0)
-			(type default)
-		)
-	)
-	(wire
-		(pts
 			(xy 254 107.95) (xy 266.7 107.95)
 		)
@@
 	(wire
 		(pts
-			(xy 57.15 138.43) (xy 57.15 140.97)
-		)
-		(stroke
-			(width 0)
-			(type default)
-		)
-	)
-	(wire
-		(pts
 			(xy 156.21 104.14) (xy 156.21 110.49)
 		)
@@
 	(wire
 		(pts
-			(xy 57.15 113.03) (xy 57.15 115.57)
-		)
-		(stroke
-			(width 0)
-			(type default)
-		)
-	)
-	(wire
-		(pts
 			(xy 207.01 59.69) (xy 207.01 58.42)
 		)
@@
 	(wire
 		(pts
-			(xy 57.15 130.81) (xy 57.15 133.35)
-		)
-		(stroke
-			(width 0)
-			(type default)
-		)
-	)
-	(wire
-		(pts
 			(xy 66.04 90.17) (xy 76.2 90.17)
 		)
@@
 		(pts
 			(xy 266.7 118.11) (xy 254 118.11)
-		)
-		(stroke
-			(width 0)
-			(type default)
-		)
-	)
-	(wire
-		(pts
-			(xy 57.15 140.97) (xy 57.15 143.51)
-		)
-		(stroke
-			(width 0)
-			(type default)
-		)
-	)
-	(wire
-		(pts
-			(xy 57.15 115.57) (xy 57.15 118.11)
 		)
 		(stroke
@@
 	(symbol
 		(lib_id "MCU_Microchip_ATmega:ATmega8-16P")
-		(at 41.91 140.97 0)
+		(at 49.53 151.13 0)
 		(unit 1)
 		(body_style 1)
@@
 		(fields_autoplaced yes)
 		(property "Reference" "U2"
-			(at 46.5933 102.87 0)
+			(at 54.2133 113.03 0)
 			(show_name no)
 			(do_not_autoplace no)
@@
 		)
 		(property "Value" "ATmega8-16P"
-			(at 46.5933 105.41 0)
+			(at 54.2133 115.57 0)
 			(show_name no)
 			(do_not_autoplace no)
@@
 		)
 		(property "Footprint" "Package_DIP:DIP-28_W7.62mm"
-			(at 41.91 140.97 0)
+			(at 49.53 151.13 0)
 			(hide yes)
 			(show_name no)
@@
 		)
 		(property "Datasheet" "http://ww1.microchip.com/downloads/en/DeviceDoc/atmel-2486-8-bit-avr-microcontroller-atmega8_l_datasheet.pdf"
-			(at 41.91 140.97 0)
+			(at 49.53 151.13 0)
 			(hide yes)
 			(show_name no)
@@
 		)
 		(property "Description" "16MHz, 8kB Flash, 1kB SRAM, 512B EEPROM, DIP-28"
-			(at 41.91 140.97 0)
+			(at 49.53 151.13 0)
 			(hide yes)
 			(show_name no)

Commit message: merging scripts
Parts:
- removed U2: ATmega8-16P, Package_DIP:DIP-28_W7.62mm, symbol MCU_Microchip_ATmega:ATmega8-16P
Connections:
- no-connect marks 28 -> 0
Changed lines of the file:
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@@
 		(color 0 0 0 0)
-	)
-	(no_connect
-		(at 64.77 148.59)
-	)
-	(no_connect
-		(at 34.29 123.19)
-	)
-	(no_connect
-		(at 64.77 123.19)
-	)
-	(no_connect
-		(at 64.77 158.75)
-	)
-	(no_connect
-		(at 34.29 128.27)
-	)
-	(no_connect
-		(at 64.77 166.37)
-	)
-	(no_connect
-		(at 64.77 130.81)
-	)
-	(no_connect
-		(at 64.77 173.99)
-	)
-	(no_connect
-		(at 34.29 138.43)
-	)
-	(no_connect
-		(at 64.77 161.29)
-	)
-	(no_connect
-		(at 64.77 135.89)
-	)
-	(no_connect
-		(at 64.77 153.67)
-	)
-	(no_connect
-		(at 64.77 163.83)
-	)
-	(no_connect
-		(at 64.77 176.53)
-	)
-	(no_connect
-		(at 52.07 115.57)
-	)
-	(no_connect
-		(at 64.77 128.27)
-	)
-	(no_connect
-		(at 49.53 186.69)
-	)
-	(no_connect
-		(at 64.77 151.13)
-	)
-	(no_connect
-		(at 34.29 133.35)
-	)
-	(no_connect
-		(at 64.77 140.97)
-	)
-	(no_connect
-		(at 64.77 125.73)
-	)
-	(no_connect
-		(at 64.77 143.51)
-	)
-	(no_connect
-		(at 52.07 186.69)
-	)
-	(no_connect
-		(at 64.77 146.05)
-	)
-	(no_connect
-		(at 64.77 168.91)
-	)
-	(no_connect
-		(at 64.77 133.35)
-	)
-	(no_connect
-		(at 64.77 171.45)
-	)
-	(no_connect
-		(at 49.53 115.57)
 	)
 	(wire
@@
 					(unit 1)
 				)
-			)
-		)
-	)
-	(symbol
-		(lib_id "MCU_Microchip_ATmega:ATmega8-16P")
-		(at 49.53 151.13 0)
-		(unit 1)
-		(body_style 1)
-		(exclude_from_sim no)
-		(in_bom yes)
-		(on_board yes)
-		(in_pos_files yes)
-		(dnp no)
-		(fields_autoplaced yes)
-		(property "Reference" "U2"
-			(at 54.2133 113.03 0)
-			(show_name no)
-			(do_not_autoplace no)
-			(effects
-				(font
-					(size 1.27 1.27)
-				)
-				(justify left)
-			)
-		)
-		(property "Value" "ATmega8-16P"
-			(at 54.2133 115.57 0)
-			(show_name no)
-			(do_not_autoplace no)
-			(effects
-				(font
-					(size 1.27 1.27)
-				)
-				(justify left)
-			)
-		)
-		(property "Footprint" "Package_DIP:DIP-28_W7.62mm"
-			(at 49.53 151.13 0)
-			(hide yes)
-			(show_name no)
-			(do_not_autoplace no)
-			(effects
-				(font
-					(size 1.27 1.27)
-					(italic yes)
-				)
-			)
-		)
-		(property "Datasheet" "http://ww1.microchip.com/downloads/en/DeviceDoc/atmel-2486-8-bit-avr-microcontroller-atmega8_l_datasheet.pdf"
-			(at 49.53 151.13 0)
-			(hide yes)
-			(show_name no)
-			(do_not_autoplace no)
-			(effects
-				(font
-					(size 1.27 1.27)
-				)
-			)
-		)
-		(property "Description" "16MHz, 8kB Flash, 1kB SRAM, 512B EEPROM, DIP-28"
-			(at 49.53 151.13 0)
-			(hide yes)
-			(show_name no)
-			(do_not_autoplace no)
-			(effects
-				(font
-					(size 1.27 1.27)
-				)
-			)
-		)
-		(pin "13"
-		)
-		(pin "15"
-		)
-		(pin "2"
-		)
-		(pin "4"
-		)
-		(pin "12"
-		)
-		(pin "14"
-		)
-		(pin "22"
-		)
-		(pin "23"
-		)
-		(pin "16"
-		)
-		(pin "18"
-		)
-		(pin "9"
-		)
-		(pin "5"
-		)
-		(pin "19"
-		)
-		(pin "20"
-		)
-		(pin "10"
-		)
-		(pin "8"
-		)
-		(pin "6"
-		)
-		(pin "11"
-		)
-		(pin "21"
-		)
-		(pin "7"
-		)
-		(pin "27"
-		)
-		(pin "28"
-		)
-		(pin "25"
-		)
-		(pin "26"
-		)
-		(pin "3"
-		)
-		(pin "17"
-		)
-		(pin "1"
-		)
-		(pin "24"
-		)
-		(instances
-			(project "ktest"
-				(path "/f14ff7c3-fe34-4697-84b8-3cc06a5a3565"
-					(reference "U2")
-					(unit 1)
-				)
