File: ktest.kicad_sch (KiCad schematic)
At the start: 40 parts, among them J1 Conn_01x03_Pin

Commit message: detailing schematic
Parts:
- removed C1, C2, C3: 10n, Capacitor_SMD:CP_Elec_5x5.9, symbol Device:C
- removed C10: 6p, Capacitor_SMD:C_0603_1608Metric_Pad1.08x0.95mm_HandSolder, symbol Device:C
- removed C11: 9p, Capacitor_SMD:C_0603_1608Metric_Pad1.08x0.95mm_HandSolder, symbol Device:C
- removed C12: 5p, Capacitor_SMD:C_0603_1608Metric_Pad1.08x0.95mm_HandSolder, symbol Device:C
- removed C13: 8p, Capacitor_SMD:C_0603_1608Metric_Pad1.08x0.95mm_HandSolder, symbol Device:C
- removed C14: 10p, Capacitor_SMD:C_0603_1608Metric_Pad1.08x0.95mm_HandSolder, symbol Device:C
- removed C15: 11p, Capacitor_SMD:C_0603_1608Metric_Pad1.08x0.95mm_HandSolder, symbol Device:C
- removed C16: 12p, Capacitor_SMD:C_0603_1608Metric_Pad1.08x0.95mm_HandSolder, symbol Device:C
- removed C17: 16p, Capacitor_SMD:C_0603_1608Metric_Pad1.08x0.95mm_HandSolder, symbol Device:C
- removed C18: 15p, Capacitor_SMD:C_0603_1608Metric_Pad1.08x0.95mm_HandSolder, symbol Device:C
- removed C19: 14p, Capacitor_SMD:C_0603_1608Metric_Pad1.08x0.95mm_HandSolder, symbol Device:C
- removed C20: 13p, Capacitor_SMD:C_0603_1608Metric_Pad1.08x0.95mm_HandSolder, symbol Device:C
- removed C5: 1p, Capacitor_SMD:C_0603_1608Metric_Pad1.08x0.95mm_HandSolder, symbol Device:C
- removed C6: 2p, Capacitor_SMD:C_0603_1608Metric_Pad1.08x0.95mm_HandSolder, symbol Device:C
- removed C7: 3p, Capacitor_SMD:C_0603_1608Metric_Pad1.08x0.95mm_HandSolder, symbol Device:C
- removed C8: 4p, Capacitor_SMD:C_0603_1608Metric_Pad1.08x0.95mm_HandSolder, symbol Device:C
- removed C9: 7p, Capacitor_SMD:C_0603_1608Metric_Pad1.08x0.95mm_HandSolder, symbol Device:C
- removed D1: LED, LED_THT:LED_D1.8mm_W3.3mm_H2.4mm, symbol Device:LED
- removed H1, H2: MountingHole, MountingHole:MountingHole_3.2mm_M3, symbol Mechanical:MountingHole
- removed H3: MountingHole, MountingHole:MountingHole_2.7mm_M2.5, symbol Mechanical:MountingHole
- removed J1: Conn_01x03_Pin, Connector_PinSocket_2.54mm:PinSocket_1x03_P2.54mm_Vertical, symbol Connector:Conn_01x03_Pin
- removed R1, R2, R3, R6, R7: 10k, Resistor_SMD:R_01005_0402Metric, symbol Device:R
- removed R11: 1k, Resistor_SMD:R_0805_2012Metric_Pad1.20x1.40mm_HandSolder, symbol Device:R
- removed R12: 2k2, Resistor_SMD:R_0805_2012Metric_Pad1.20x1.40mm_HandSolder, symbol Device:R
- removed R13: 3k3, Resistor_SMD:R_0805_2012Metric_Pad1.20x1.40mm_HandSolder, symbol Device:R
- removed R14: 4k7, Resistor_SMD:R_0805_2012Metric_Pad1.20x1.40mm_HandSolder, symbol Device:R
- removed R15: 5k1, Resistor_SMD:R_0805_2012Metric_Pad1.20x1.40mm_HandSolder, symbol Device:R
- removed R16: 5k6, Resistor_SMD:R_0805_2012Metric_Pad1.20x1.40mm_HandSolder, symbol Device:R
- removed R17: 6k8, Resistor_SMD:R_0805_2012Metric_Pad1.20x1.40mm_HandSolder, symbol Device:R
- removed R18: 7k5, Resistor_SMD:R_0805_2012Metric_Pad1.20x1.40mm_HandSolder, symbol Device:R
- removed R19: 9k1, Resistor_SMD:R_0805_2012Metric_Pad1.20x1.40mm_HandSolder, symbol Device:R
- removed R4, R5: 10k, Resistor_THT:R_Axial_DIN0414_L11.9mm_D4.5mm_P5.08mm_Vertical, symbol Device:R
Other:
- sheet child_1 renamed System_overview
- sheet System_overview: file child_1.kicad_sch -> System_overview.kicad_sch
- sheet System_overview ports: added none; removed a, n

Commit message: testing links
Other:
- note added: "${PROJECT}"
- note added: "${SHEET_NAME_5}"
- note added: "${SHEET_NAME_6}"
- note added: "${SHEET_NAME_7}"
- note added: "${SHEET_NAME_8}"
- note added: "${SHEET_TITLE_1}"
- note added: "${SHEET_TITLE_2}"
- note added: "${SHEET_TITLE_3}"
- note added: "${SHEET_TITLE_4}"
- note added: "Page"
- note added: "Table of contents"

Commit message: system overview and interfaces done
Other:
- sheet System_overview renamed System overview
- note added: "07/10/2026"
- note added: "08/10/2026"
- note added: "1"
- note added: "1.0.0"
- note added: "2"
- note added: "3"
- note added: "4"
- note added: "5"
- note added: "6"
- note added: "7"
- note added: "8"
- note added: "Change history"
- note added: "First release"
- note added: "Fix R1234 value due to issue xyz etc etc etc. Update C14 to 10 nF to reduce roll-off frequency."
- note added: "TBD"
- note removed: "Page"

Commit message: testing green mask
Changed lines of the file:
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@@
 				(face "DejaVu Sans")
 				(size 5.08 5.08)
-				(thickness 0.3175)
 				(color 0 0 0 1)
 			)

Commit message: testing blue mask
Other:
- note removed: "${SHEET_NAME_5}"
- note removed: "${SHEET_NAME_6}"
- note removed: "${SHEET_NAME_7}"
- note removed: "${SHEET_NAME_8}"

Commit message: sch2
Other:
- note added: "10"
- note added: "11"
- note added: "12"
- note added: "9"
Changed lines of the file:
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@@
+		)
+	)
+	(text "9"
+		(exclude_from_sim no)
+		(at 26.035 80.01 0)
+		(effects
+			(font
+				(face "DejaVu Sans")
+				(size 2.032 2.032)
+				(thickness 0.3175)
+				(color 0 0 0 1)
+			)
+			(justify left top)
 		)
 	)
@@
 		)
 	)
+	(text "12"
+		(exclude_from_sim no)
+		(at 26.035 95.25 0)
+		(effects
+			(font
+				(face "DejaVu Sans")
+				(size 2.032 2.032)
+				(thickness 0.3175)
+				(color 0 0 0 1)
+			)
+			(justify left top)
+		)
+	)
 	(text "2"
 		(exclude_from_sim no)
@@
 		)
 	)
+	(text "10"
+		(exclude_from_sim no)
+		(at 26.035 85.09 0)
+		(effects
+			(font
+				(face "DejaVu Sans")
+				(size 2.032 2.032)
+				(thickness 0.3175)
+				(color 0 0 0 1)
+			)
+			(justify left top)
+		)
+	)
+	(text "11"
+		(exclude_from_sim no)
+		(at 26.035 90.17 0)
+		(effects
+			(font
+				(face "DejaVu Sans")
+				(size 2.032 2.032)
+				(thickness 0.3175)
+				(color 0 0 0 1)
+			)
+			(justify left top)
+		)
+	)
 	(text "Fix R1234 value due to issue xyz etc etc etc. Update C14 to 10 nF to reduce roll-off frequency."
 		(exclude_from_sim no)
@@
 	)
 	(sheet
-		(at 25.4 165.1)
+		(at 88.9 165.1)
 		(size 38.1 25.4)
 		(exclude_from_sim no)
@@
 		)
 		(property "Sheetname" "System overview"
-			(at 25.4 164.3884 0)
+			(at 88.9 164.3884 0)
 			(show_name no)
 			(do_not_autoplace no)
@@
 		)
 		(property "Sheetfile" "System_overview.kicad_sch"
-			(at 25.4 191.0846 0)
+			(at 88.9 191.0846 0)
 			(show_name no)
 			(do_not_autoplace no)

Commit message: reorganised sch and pcb
Other:
- note added: "${SHEET_TITLE_10}"
- note added: "${SHEET_TITLE_11}"
- note added: "${SHEET_TITLE_12}"
- note added: "${SHEET_TITLE_5}"
- note added: "${SHEET_TITLE_6}"
- note added: "${SHEET_TITLE_7}"
- note added: "${SHEET_TITLE_8}"
- note added: "${SHEET_TITLE_9}"
- title: 1 kV strobe -> Root_sch
Changed lines of the file:
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@@
 	(paper "A4")
 	(title_block
-		(title "1 kV strobe")
+		(title "Root_sch")
 		(date "2026-10-06")
 		(rev "0.0.1")
@@
 		)
 	)
+	(text "${SHEET_TITLE_7}"
+		(exclude_from_sim no)
+		(at 32.385 69.85 0)
+		(effects
+			(font
+				(face "DejaVu Sans")
+				(size 2.032 2.032)
+				(thickness 0.3175)
+				(color 0 0 0 1)
+			)
+			(justify left top)
+			(href "#7")
+		)
+	)
+	(text "${SHEET_TITLE_8}"
+		(exclude_from_sim no)
+		(at 32.385 74.93 0)
+		(effects
+			(font
+				(face "DejaVu Sans")
+				(size 2.032 2.032)
+				(thickness 0.3175)
+				(color 0 0 0 1)
+			)
+			(justify left top)
+			(href "#8")
+		)
+	)
 	(text "${SHEET_TITLE_3}"
 		(exclude_from_sim no)
@@
 		)
 	)
+	(text "${SHEET_TITLE_9}"
+		(exclude_from_sim no)
+		(at 32.385 80.01 0)
+		(effects
+			(font
+				(face "DejaVu Sans")
+				(size 2.032 2.032)
+				(thickness 0.3175)
+				(color 0 0 0 1)
+			)
+			(justify left top)
+			(href "#9")
+		)
+	)
 	(text "1.0.0"
 		(exclude_from_sim no)
@@
 		)
 	)
+	(text "${SHEET_TITLE_5}"
+		(exclude_from_sim no)
+		(at 32.385 59.69 0)
+		(effects
+			(font
+				(face "DejaVu Sans")
+				(size 2.032 2.032)
+				(thickness 0.3175)
+				(color 0 0 0 1)
+			)
+			(justify left top)
+			(href "#5")
+		)
+	)
 	(text "TBD"
 		(exclude_from_sim no)
@@
 		)
 	)
+	(text "${SHEET_TITLE_10}"
+		(exclude_from_sim no)
+		(at 32.385 85.09 0)
+		(effects
+			(font
+				(face "DejaVu Sans")
+				(size 2.032 2.032)
+				(thickness 0.3175)
+				(color 0 0 0 1)
+			)
+			(justify left top)
+			(href "#10")
+		)
+	)
 	(text "8"
 		(exclude_from_sim no)
@@
 		)
 	)
+	(text "${SHEET_TITLE_6}"
+		(exclude_from_sim no)
+		(at 32.385 64.77 0)
+		(effects
+			(font
+				(face "DejaVu Sans")
+				(size 2.032 2.032)
+				(thickness 0.3175)
+				(color 0 0 0 1)
+			)
+			(justify left top)
+			(href "#6")
+		)
+	)
 	(text "07/10/2026"
 		(exclude_from_sim no)
@@
 		)
 	)
+	(text "${SHEET_TITLE_11}"
+		(exclude_from_sim no)
+		(at 32.385 90.17 0)
+		(effects
+			(font
+				(face "DejaVu Sans")
+				(size 2.032 2.032)
+				(thickness 0.3175)
+				(color 0 0 0 1)
+			)
+			(justify left top)
+			(href "#11")
+		)
+	)
+	(text "${SHEET_TITLE_12}"
+		(exclude_from_sim no)
+		(at 32.385 95.25 0)
+		(effects
+			(font
+				(face "DejaVu Sans")
+				(size 2.032 2.032)
+				(thickness 0.3175)
+				(color 0 0 0 1)
+			)
+			(justify left top)
+			(href "#12")
+		)
+	)
 	(text "3"
 		(exclude_from_sim no)
@@
 		)
 	)
+	(polyline
+		(pts
+			(xy 86.36 176.53) (xy 184.15 176.53)
+		)
+		(stroke
+			(width 0)
+			(type default)
+		)
+	)
+	(polyline
+		(pts
+			(xy 86.36 33.02) (xy 86.36 196.85)
+		)
+		(stroke
+			(width 0)
+			(type default)
+		)
+	)
 	(sheet
-		(at 88.9 165.1)
-		(size 38.1 25.4)
+		(at 88.9 180.34)
+		(size 38.1 12.7)
 		(exclude_from_sim no)
 		(in_bom yes)
@@
 		)
 		(property "Sheetname" "System overview"
-			(at 88.9 164.3884 0)
+			(at 88.9 179.6284 0)
 			(show_name no)
 			(do_not_autoplace no)
@@
 		)
 		(property "Sheetfile" "System_overview.kicad_sch"
-			(at 88.9 191.0846 0)
+			(at 88.9 193.6246 0)
 			(show_name no)
 			(do_not_autoplace no)
