File: Block_diagram.kicad_sch (KiCad schematic)
At the start: 46 parts, among them J2 Conn_01x03_Pin, U1 STM32WBA55HEFx

Commit message: creating hierarchy
Parts:
- renumbered C4 to C1, C14 to C11, C18 to C12, C7 to C13, C11 to C14, C19 to C16, C8 to C17, C12 to C18, C16 to C19, C21 to C2, C22 to C3, C23 to C4, C9 to C6, C13 to C7, C17 to C8, C6 to C9, D2 to D1, D3 to D2, H4 to H1, H5 to H2, H6 to H3, J2 to J1, R8 to R1, R26 to R10, R27 to R11, R28 to R12, R29 to R13, R30 to R14, R31 to R15, R32 to R16, R33 to R17, R34 to R18, R35 to R19, R20 to R2, R21 to R3, R9 to R4, R10 to R5, R22 to R6, R23 to R7, R24 to R8, R25 to R9
Other:
- added sheet child_1 (child_1.kicad_sch)

Commit message: testing links
Other:
- note added: "Top page"
Changed lines of the file:
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@@
 	(generator_version "10.0")
 	(paper "A4")
+	(text "Top page"
+		(exclude_from_sim no)
+		(at 12.7 196.85 0)
+		(effects
+			(font
+				(face "DejaVu Sans")
+				(size 2.032 2.032)
+				(thickness 0.3175)
+				(color 0 0 0 1)
+			)
+			(justify left bottom)
+			(href "#1")
+		)
+	)
 	(junction
 		(at 140.97 135.89)

Commit message: system overview and interfaces done
Parts:
- removed C1, C2, C3, C4: 10n, Capacitor_SMD:CP_Elec_5x5.9, symbol Device:C
- removed C10: 6p, Capacitor_SMD:C_0603_1608Metric_Pad1.08x0.95mm_HandSolder, symbol Device:C
- removed C11: 10p, Capacitor_SMD:C_0603_1608Metric_Pad1.08x0.95mm_HandSolder, symbol Device:C
- removed C12: 15p, Capacitor_SMD:C_0603_1608Metric_Pad1.08x0.95mm_HandSolder, symbol Device:C
- removed C13: 3p, Capacitor_SMD:C_0603_1608Metric_Pad1.08x0.95mm_HandSolder, symbol Device:C
- removed C14: 9p, Capacitor_SMD:C_0603_1608Metric_Pad1.08x0.95mm_HandSolder, symbol Device:C
- removed C15: 11p, Capacitor_SMD:C_0603_1608Metric_Pad1.08x0.95mm_HandSolder, symbol Device:C
- removed C16: 14p, Capacitor_SMD:C_0603_1608Metric_Pad1.08x0.95mm_HandSolder, symbol Device:C
- removed C17: 4p, Capacitor_SMD:C_0603_1608Metric_Pad1.08x0.95mm_HandSolder, symbol Device:C
- removed C18: 5p, Capacitor_SMD:C_0603_1608Metric_Pad1.08x0.95mm_HandSolder, symbol Device:C
- removed C19: 12p, Capacitor_SMD:C_0603_1608Metric_Pad1.08x0.95mm_HandSolder, symbol Device:C
- removed C20: 13p, Capacitor_SMD:C_0603_1608Metric_Pad1.08x0.95mm_HandSolder, symbol Device:C
- removed C5: 1p, Capacitor_SMD:C_0603_1608Metric_Pad1.08x0.95mm_HandSolder, symbol Device:C
- removed C6: 7p, Capacitor_SMD:C_0603_1608Metric_Pad1.08x0.95mm_HandSolder, symbol Device:C
- removed C7: 8p, Capacitor_SMD:C_0603_1608Metric_Pad1.08x0.95mm_HandSolder, symbol Device:C
- removed C8: 16p, Capacitor_SMD:C_0603_1608Metric_Pad1.08x0.95mm_HandSolder, symbol Device:C
- removed C9: 2p, Capacitor_SMD:C_0603_1608Metric_Pad1.08x0.95mm_HandSolder, symbol Device:C
- removed D1, D2: LED, LED_THT:LED_D1.8mm_W3.3mm_H2.4mm, symbol Device:LED
- removed H1, H2: MountingHole, MountingHole:MountingHole_3.2mm_M3, symbol Mechanical:MountingHole
- removed H3: MountingHole, MountingHole:MountingHole_2.7mm_M2.5, symbol Mechanical:MountingHole
- removed J1: Conn_01x03_Pin, Connector_PinSocket_2.54mm:PinSocket_1x03_P2.54mm_Vertical, symbol Connector:Conn_01x03_Pin
- removed R1, R2, R3, R6, R7, R8: 10k, Resistor_SMD:R_01005_0402Metric, symbol Device:R
- removed R10, R4, R5, R9: 10k, Resistor_THT:R_Axial_DIN0414_L11.9mm_D4.5mm_P5.08mm_Vertical, symbol Device:R
- removed R11: 1k, Resistor_SMD:R_0805_2012Metric_Pad1.20x1.40mm_HandSolder, symbol Device:R
- removed R12: 4k7, Resistor_SMD:R_0805_2012Metric_Pad1.20x1.40mm_HandSolder, symbol Device:R
- removed R13: 6k8, Resistor_SMD:R_0805_2012Metric_Pad1.20x1.40mm_HandSolder, symbol Device:R
- removed R14: 2k2, Resistor_SMD:R_0805_2012Metric_Pad1.20x1.40mm_HandSolder, symbol Device:R
- removed R15: 5k1, Resistor_SMD:R_0805_2012Metric_Pad1.20x1.40mm_HandSolder, symbol Device:R
- removed R16: 7k5, Resistor_SMD:R_0805_2012Metric_Pad1.20x1.40mm_HandSolder, symbol Device:R
- removed R17: 3k3, Resistor_SMD:R_0805_2012Metric_Pad1.20x1.40mm_HandSolder, symbol Device:R
- removed R18: 5k6, Resistor_SMD:R_0805_2012Metric_Pad1.20x1.40mm_HandSolder, symbol Device:R
- removed R19: 9k1, Resistor_SMD:R_0805_2012Metric_Pad1.20x1.40mm_HandSolder, symbol Device:R
- removed U1: STM32WBA55HEFx, Package_CSP:ST_WLCSP-41_2.98x2.76mm_Layout13x7_P0.4mm_Stagger, symbol MCU_ST_STM32WB:STM32WBA55HEFx
Connections:
- no-connect marks 1 -> 0
Other:
- removed sheet child_1
- note added: "${SHEETNAME}"
- note added: "Return to front sheet"
- note removed: "Top page"

Commit message: testing green mask
Parts:
- added C1, C13, C19, C20, C25, C6, C9: 100n, Capacitor_SMD:C_0603_1608Metric_Pad1.08x0.95mm_HandSolder, symbol Device:C
- added C10, C14: 22p, Capacitor_SMD:C_0603_1608Metric_Pad1.08x0.95mm_HandSolder, symbol Device:C
- added C11, C16: 1u, Capacitor_SMD:C_0603_1608Metric_Pad1.08x0.95mm_HandSolder, symbol Device:C
- added C12: 33p, Capacitor_SMD:C_0603_1608Metric_Pad1.08x0.95mm_HandSolder, symbol Device:C
- added C15, C17, C18: 22u, Capacitor_SMD:C_1210_3225Metric_Pad1.33x2.70mm_HandSolder, symbol Device:C
- added C2, C4: 4.7u, Capacitor_SMD:C_1206_3216Metric_Pad1.33x1.80mm_HandSolder, symbol Device:C
- added C21, C22, C23, C7, C8: 1n, Capacitor_SMD:C_0603_1608Metric_Pad1.08x0.95mm_HandSolder, symbol Device:C
- added C24: 220u, Capacitor_SMD:CP_Elec_10x10, symbol Device:C_Polarized
- added C26, C27, C3, C5: 10n, Capacitor_SMD:C_0603_1608Metric_Pad1.08x0.95mm_HandSolder, symbol Device:C
- added D1: BAV99, Package_TO_SOT_SMD:SOT-23, symbol Diode:BAV99
- added J1: JST B4B XH A, Connector_JST:JST_XH_B4B-XH-A_1x04_P2.50mm_Vertical, symbol Connector:Conn_01x04_Pin
- added J10, J7, J9: JST B6B XH A, Connector_JST:JST_XH_B6B-XH-A_1x06_P2.50mm_Vertical, symbol Connector:Conn_01x06_Pin
- added J2: 2.54 mm header, Connector_PinHeader_2.54mm:PinHeader_1x04_P2.54mm_Vertical, symbol Connector:Conn_01x04_Pin
- added J3: Conn_01x14_Pin, Connector_PinSocket_2.54mm:PinSocket_1x14_P2.54mm_Vertical, symbol Connector:Conn_01x14_Pin
- added J4: HX JN1.27-2x5 WZ H4.9, Personal:JN1.27-2x5 WZ H4.9, symbol Connector_Generic:Conn_02x05_Odd_Even
- added J5: USB_C_Receptacle_USB2.0_16P, Personal:USB_C_socket_16P_vertical, symbol Connector:USB_C_Receptacle_USB2.0_16P
- added J6: Dell DC jack, Personal:Dell DC jack, symbol personal:Dell_DC_barrel_jack
- added J8: DC barrel assy, Personal:Dell_barrel_assy, symbol personal:DC_barrel_assy
- added JP1, JP10, JP11, JP12, JP13, JP15, JP16, JP17, JP2, JP21, JP3, JP8: 0R, Personal:Jumper_0603, symbol Device:R
- added JP14, JP19, JP4, JP5, JP7: 0R, Resistor_SMD:R_1206_3216Metric_Pad1.30x1.75mm_HandSolder, symbol Device:R
- added JP18, JP22: 0R, Resistor_THT:R_Axial_DIN0204_L3.6mm_D1.6mm_P7.62mm_Horizontal, symbol Device:R
- added JP20, JP6: 0R, Resistor_SMD:R_0603_1608Metric_Pad0.98x0.95mm_HandSolder, symbol Device:R
- added JP9: 0R, Resistor_THT:R_Axial_DIN0204_L3.6mm_D1.6mm_P5.08mm_Horizontal, symbol Device:R
- added L1: 10u, Personal:L_Bourns_SRP6540, symbol Device:L
- added P1, P12, P13, P15, P16, P2, P22, P25, P27, P28, P30, P31, P32, P33, P43, P44, P45, P47, P6: (no value), symbol personal:Cosmetic_OUT
- added P10, P11, P14, P17, P18, P19, P20, P21, P23, P24, P26, P29, P3, P37, P38, P39, P4, P40, P41, P42, P5, P7, P8, P9: (no value), symbol personal:Cosmetic_IN
- added P34, P35, P36, P46, P48, P49: (no value), symbol personal:Cosmetic_IO
- added R1, R2, R7, R8, R9: 10k, Resistor_SMD:R_0603_1608Metric_Pad0.98x0.95mm_HandSolder, symbol Device:R
- added R10, R12, R13, R4, R5: 2k2, Resistor_SMD:R_0603_1608Metric_Pad0.98x0.95mm_HandSolder, symbol Device:R
- added R11: 820, Resistor_SMD:R_0603_1608Metric_Pad0.98x0.95mm_HandSolder, symbol Device:R
- added R14, R15: 5k1, Resistor_SMD:R_0603_1608Metric_Pad0.98x0.95mm_HandSolder, symbol Device:R
- added R3: 64.9k, Resistor_SMD:R_0603_1608Metric_Pad0.98x0.95mm_HandSolder, symbol Device:R
- added R6: 23.2k, Resistor_SMD:R_0603_1608Metric_Pad0.98x0.95mm_HandSolder, symbol Device:R
- added TFT1: TFT_2.4in_320x240, Personal:Display_240x320_ILI9341_2.4in_no_pads, symbol personal:TFT_2.8_IN_320x240
- added TP1, TP10, TP11, TP12, TP13, TP14, TP15, TP16, TP17, TP18, TP19, TP2, TP20, TP21, TP3, TP4, TP5, TP6, TP7, TP8, TP9: TestPoint, TestPoint:TestPoint_THTPad_D1.0mm_Drill0.5mm, symbol Connector:TestPoint
- added U1: LMR380x0, Package_SO:Texas_HSOP-8-1EP_3.9x4.9mm_P1.27mm_ThermalVias, symbol personal:LMR380x0
- added U2: STM32G431K8Tx, Package_QFP:LQFP-32_7x7mm_P0.8mm, symbol MCU_ST_STM32G4:STM32G431K8Tx
- added U3: VNH7070, Package_SO:JEITA_SOIC-16_3.9x9.9mm_P1.27mm, symbol personal:VNH7070
- added U4: USBLC6-2SC6, Package_TO_SOT_SMD:SOT-23-6, symbol Power_Protection:USBLC6-2SC6
- added Y1: 20 MHz, Crystal:Crystal_SMD_3225-4Pin_3.2x2.5mm_HandSoldering, symbol Device:Crystal_GND24_Small
Connections:
- new net: J3.12 (Pin_12), JP3.2
- new net: J3.11 (Pin_11), JP4.2
- new net: J5.A4 (VBUS), J5.A9 (VBUS), J5.B4 (VBUS), J5.B9 (VBUS), TP16.1
- new net: J3.14 (Pin_14), JP1.2
- new net: C9.1, U1.7 (BOOT)
- new net: J3.10 (Pin_10), JP5.2
- new net: J3.13 (Pin_13), JP2.2
- new net: J3.3 (Pin_3), JP11.2
- new net: J3.4 (Pin_4), JP10.2
- new net: J3.5 (Pin_5), JP9.2
- new net: J3.6 (Pin_6), JP8.2
- new net: J3.7 (Pin_7), JP7.2
- new net: J3.9 (Pin_9), JP6.2
- new net: JP19.1, R10.2, R11.1
- new net: J10.1 (Pin_1), J9.1 (Pin_1)
- new net: J10.2 (Pin_2), J9.2 (Pin_2)
- new net: J10.3 (Pin_3), J9.3 (Pin_3)
- new net: J10.4 (Pin_4), J9.4 (Pin_4)
- new net: J10.5 (Pin_5), J9.5 (Pin_5)
- new net: J10.6 (Pin_6), J9.6 (Pin_6)
- new net 3V3_REG: C12.1, C15.1, C17.1, C18.1, JP12.1, L1.2, R6.1, TP7.1
- new net BOOT0: R9.1, TP9.1, U2.31 (PB8)
- new net BOT_EOT: C3.1, J1.1 (Pin_1), R1.2, R5.1
- new net BOT_filt: C7.1, P13.1, P32.1, R5.2, TP4.1, U2.19 (PA9)
- new net CC1: J5.A5 (CC1), R14.1
- new net CC2: J5.B5 (CC2), R15.1
- new net CS': JP19.2, TP15.1, U3.13 (CS)
- new net D+: J5.A6 (D+), J5.B6 (D+), JP21.1
- new net D+': JP21.2, U4.6 (I/O1)
- new net D-: J5.A7 (D-), J5.B7 (D-), JP20.1
- new net D-': JP20.2, U4.4 (I/O2)
- new net DISP_CS: JP11.1, P11.1, P31.1, U2.18 (PA8)
- new net DISP_DC: JP9.1, P27.1, P9.1, U2.9 (PA4)
- new net DISP_MISO: JP2.1, JP6.1, P2.1, P29.1, P6.1, U2.11 (PA6)
- new net DISP_MOSI: JP3.1, JP8.1, P3.1, P30.1, P8.1, U2.12 (PA7)
- new net DISP_RST: JP10.1, P10.1, P15.1, U2.13 (PB0)
- new net DISP_SCK: JP5.1, JP7.1, P28.1, P5.1, P7.1, U2.10 (PA5)
- new net ENCa: C27.1, J7.5 (Pin_5), R12.2
- new net ENCa_filt: C23.1, P19.1, P44.1, R12.1, TP12.1, U2.29 (PB6)
- new net ENCb: C26.1, J7.6 (Pin_6), R13.2
- new net ENCb_filt: C22.1, P20.1, P45.1, R13.1, TP13.1, U2.30 (PB7)
- new net FB: C12.2, R6.2, R7.1, TP5.1, U1.5 (FB)
- new net GND: C1.2, C10.2, C11.2, C13.2, C14.2, C15.2, C16.2, C17.2, C18.2, C19.2, C2.2, C20.2, C21.2, C22.2, C23.2, C24.2, C25.2, C26.2, C27.2, C3.2, C4.2, C5.2, C6.2, C7.2, C8.2, D1.1 (K), J1.2 (Pin_2), J1.3 (Pin_3), J3.2 (Pin_2), J4.5 (Pin_5), J4.6 (Pin_6), J5.A1 (GND), J5.A12 (GND), J5.B1 (GND), J5.B12 (GND), J5.SH (SHIELD), J7.4 (Pin_4), J8.2 (-), R11.2, R14.2, R15.2, R3.2, R7.2, R9.2, TP17.1, TP18.1, TP19.1, TP20.1, TP21.1, U1.1 (GND), U1.9 (EP), U2.14 (VSSA), U2.16 (VSS), U2.32 (VSS), U3.1 (GNDa), U3.16 (GNDa), U3.8 (GNDb), U3.9 (GNDb), U4.2 (GND), Y1.2 (G), Y1.4 (G)
- new net GND_2: J6.3 (-), J6.SH
- new net INa: JP15.1, P18.1, P39.1, U2.28 (PB5)
- new net INa': JP15.2, U3.3 (INa)
- new net INb: JP16.1, P17.1, P40.1, U2.27 (PB4)
- new net INb': JP16.2, U3.6 (INb)
- new net MOT_CS: C21.1, D1.3 (K), P23.1, P43.1, R10.1, TP14.1, U2.5 (PA0)
- new net NRST: J4.1 (Pin_1), P14.1, P22.1, R8.2, TP8.1, U2.4 (PG10)
- new net OUTa: J7.2 (Pin_2), U3.15 (OUTa), U3.2 (OUTa)
- new net OUTb: J7.1 (Pin_1), JP22.1
- new net OUTb': JP22.2, U3.10 (OUTb), U3.7 (OUTb)
- new net PG: TP1.1, U1.6 (PG)
- new net PWM: JP17.1, P38.1, P41.1, U2.25 (PA15)
- new net PWM': JP17.2, U3.11 (PWM)
- new net RT: R3.1, TP2.1, U1.4 (RT/SYNC)
- new net S19V5: C2.1, C24.1, C25.1, C4.1, C6.1, J8.1 (+), U1.2 (EN), U1.3 (VIN), U3.12 (VCC), U3.4 (VCC), U3.5 (VCC)
- new net S19V5_2: J6.1 (+)
- new net S3V3: C1.1, C11.1, C13.1, C16.1, C19.1, D1.2 (A), J3.1 (Pin_1), J3.8 (Pin_8), J4.7 (Pin_7), J4.8 (Pin_8), J7.3 (Pin_3), JP12.2, JP13.1, R1.1, R2.1, R8.1, TP10.1, U2.1 (VDD), U2.17 (VDD), U4.5 (VBUS)
- new net S3V3_A: C20.1, JP13.2, U2.15 (VDDA)
- new net SEL0: JP18.2, P24.1, P42.1, TP11.1, U2.6 (PA1)
- new net SEL0': JP18.1, U3.14 (SEL0)
- new net SW: C9.2, L1.1, TP6.1, U1.8 (SW)
- new net SWDCLK: J4.2 (Pin_2), P37.1, P47.1, U2.24 (PA14)
- new net SWDIO: J4.4 (Pin_4), P36.1, P46.1, U2.23 (PA13)
- new net SWO: JP14.1, P16.1, P21.1, U2.26 (PB3)
- new net SWO': J4.3 (Pin_3), JP14.2
- new net TCH_CS: JP4.1, P26.1, P4.1, U2.8 (PA3)
- new net TCH_IRQ: JP1.1, P1.1, P25.1, U2.7 (PA2)
- new net TOP_EOT: C5.1, J1.4 (Pin_4), R2.2, R4.1
- new net TOP_filt: C8.1, P12.1, P33.1, R4.2, TP3.1, U2.20 (PA10)
- new net USB_DM: P34.1, P49.1, U2.21 (PA11), U4.3 (I/O2)
- new net USB_DP: P35.1, P48.1, U2.22 (PA12), U4.1 (I/O1)
- new net XIN: C10.1, U2.2 (PF0), Y1.1
- new net XOUT: C14.1, U2.3 (PF1), Y1.3
- no-connect marks 0 -> 9
Other:
- note added: "3.3 V supply"
- note added: "3D model"
- note added: "Board mounting"
- note added: "End of travel switch interface"
- note added: "Microcontroller"
- note added: "Motor interface"
- note added: "SWD header"
- note added: "TFT display"
- note added: "USB interface (serial comms port)"

Commit message: testing blue mask
Parts:
- removed J10, J9: JST B6B XH A, Connector_JST:JST_XH_B6B-XH-A_1x06_P2.50mm_Vertical, symbol Connector:Conn_01x06_Pin
Changed lines of the file:
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@@
 	(wire
 		(pts
-			(xy 650.24 96.52) (xy 657.86 96.52)
-		)
-		(stroke
-			(width 0)
-			(type default)
-		)
-	)
-	(wire
-		(pts
 			(xy 542.29 114.3) (xy 542.29 115.57)
 		)
@@
 	(wire
 		(pts
-			(xy 650.24 91.44) (xy 657.86 91.44)
-		)
-		(stroke
-			(width 0)
-			(type default)
-		)
-	)
-	(wire
-		(pts
 			(xy 367.03 101.6) (xy 379.73 101.6)
 		)
@@
 	(wire
 		(pts
-			(xy 650.24 99.06) (xy 657.86 99.06)
-		)
-		(stroke
-			(width 0)
-			(type default)
-		)
-	)
-	(wire
-		(pts
 			(xy 601.98 92.71) (xy 605.79 92.71)
 		)
@@
 	(wire
 		(pts
-			(xy 650.24 101.6) (xy 657.86 101.6)
-		)
-		(stroke
-			(width 0)
-			(type default)
-		)
-	)
-	(wire
-		(pts
 			(xy 581.66 114.3) (xy 581.66 115.57)
 		)
@@
 	(wire
 		(pts
-			(xy 650.24 104.14) (xy 657.86 104.14)
-		)
-		(stroke
-			(width 0)
-			(type default)
-		)
-	)
-	(wire
-		(pts
 			(xy 401.32 82.55) (xy 401.32 85.09)
 		)
@@
 	(wire
 		(pts
-			(xy 650.24 93.98) (xy 657.86 93.98)
-		)
-		(stroke
-			(width 0)
-			(type default)
-		)
-	)
-	(wire
-		(pts
 			(xy 401.32 72.39) (xy 401.32 74.93)
 		)
@@
 	)
 	(symbol
-		(lib_id "Connector:Conn_01x06_Pin")
-		(at 662.94 96.52 0)
-		(mirror y)
-		(unit 1)
-		(body_style 1)
-		(exclude_from_sim no)
-		(in_bom yes)
-		(on_board yes)
-		(in_pos_files yes)
-		(dnp no)
-		(property "Reference" "J9"
-			(at 659.13 85.725 0)
-			(show_name no)
-			(do_not_autoplace no)
-			(effects
-				(font
-					(size 1.27 1.27)
-				)
-				(justify right)
-			)
-		)
-		(property "Value" "JST B6B XH A"
-			(at 659.13 88.265 0)
-			(show_name no)
-			(do_not_autoplace no)
-			(effects
-				(font
-					(size 1.27 1.27)
-				)
-				(justify right)
-			)
-		)
-		(property "Footprint" "Connector_JST:JST_XH_B6B-XH-A_1x06_P2.50mm_Vertical"
-			(at 662.94 96.52 0)
-			(hide yes)
-			(show_name no)
-			(do_not_autoplace no)
-			(effects
-				(font
-					(size 1.27 1.27)
-				)
-			)
-		)
-		(property "Datasheet" ""
-			(at 662.94 96.52 0)
-			(hide yes)
-			(show_name no)
-			(do_not_autoplace no)
-			(effects
-				(font
-					(size 1.27 1.27)
-				)
-			)
-		)
-		(property "Description" "Generic connector, single row, 01x06, script generated"
-			(at 662.94 96.52 0)
-			(hide yes)
-			(show_name no)
-			(do_not_autoplace no)
-			(effects
-				(font
-					(size 1.27 1.27)
-				)
-			)
-		)
-		(pin "6"
-		)
-		(pin "2"
-		)
-		(pin "3"
-		)
-		(pin "1"
-		)
-		(pin "4"
-		)
-		(pin "5"
-		)
-		(instances
-			(project "ktest"
-				(path "/f14ff7c3-fe34-4697-84b8-3cc06a5a3565/8691f566-486a-4ca4-ac00-06f17a09aade/75753c83-0606-4e75-9e41-6be2b05a7146"
-					(reference "J9")
-					(unit 1)
-				)
-			)
-		)
-	)
-	(symbol
 		(lib_id "Device:R")
 		(at 363.22 50.8 90)
@@
 					(unit 1)
 				)
-			)
-		)
-	)
-	(symbol
-		(lib_id "Connector:Conn_01x06_Pin")
-		(at 645.16 96.52 0)
-		(unit 1)
-		(body_style 1)
-		(exclude_from_sim no)
-		(in_bom yes)
-		(on_board yes)
-		(in_pos_files yes)
-		(dnp no)
-		(property "Reference" "J10"
-			(at 648.97 85.725 0)
-			(show_name no)
-			(do_not_autoplace no)
-			(effects
-				(font
-					(size 1.27 1.27)
-				)
-				(justify right)
-			)
-		)
-		(property "Value" "JST B6B XH A"
-			(at 648.97 88.265 0)
-			(show_name no)
-			(do_not_autoplace no)
-			(effects
-				(font
-					(size 1.27 1.27)
-				)
-				(justify right)
-			)
-		)
-		(property "Footprint" "Connector_JST:JST_XH_B6B-XH-A_1x06_P2.50mm_Vertical"
-			(at 645.16 96.52 0)
-			(hide yes)
-			(show_name no)
-			(do_not_autoplace no)
-			(effects
-				(font
-					(size 1.27 1.27)
-				)
-			)
-		)
-		(property "Datasheet" ""
-			(at 645.16 96.52 0)
-			(hide yes)
-			(show_name no)
-			(do_not_autoplace no)
-			(effects
-				(font
-					(size 1.27 1.27)
-				)
-			)
-		)
-		(property "Description" "Generic connector, single row, 01x06, script generated"
-			(at 645.16 96.52 0)
-			(hide yes)
-			(show_name no)
-			(do_not_autoplace no)
-			(effects
-				(font
-					(size 1.27 1.27)
-				)
-			)
-		)
-		(pin "6"
-		)
-		(pin "2"
-		)
-		(pin "3"
-		)
-		(pin "1"
-		)
-		(pin "4"
-		)
-		(pin "5"
-		)
-		(instances
-			(project "ktest"
-				(path "/f14ff7c3-fe34-4697-84b8-3cc06a5a3565/8691f566-486a-4ca4-ac00-06f17a09aade/75753c83-0606-4e75-9e41-6be2b05a7146"
-					(reference "J10")
-					(unit 1)
-				)
