File: Block_diagram.kicad_sch (KiCad schematic)
At the start: 150 parts, among them J1 JST B4B XH A, J2 2.54 mm header, J3 Conn_01x14_Pin, J4 HX JN1.27-2x5 WZ H4.9, J5 USB_C_Receptacle_USB2.0_16P, J6 Dell DC jack, J7 JST B6B XH A, J8 DC barrel assy, U1 LMR380x0, U2 STM32G431K8Tx, U3 VNH7070, U4 USBLC6-2SC6, Y1 20 MHz

Commit message: jst correction attempt
Parts:
- J2: footprint Connector_PinHeader_2.54mm:PinHeader_1x04_P2.54mm_Vertical -> Connector_PinSocket_2.54mm:PinSocket_1x04_P2.54mm_Vertical
Changed lines of the file:
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@@
 			)
 		)
-		(property "Footprint" "Connector_PinHeader_2.54mm:PinHeader_1x04_P2.54mm_Vertical"
+		(property "Footprint" "Connector_PinSocket_2.54mm:PinSocket_1x04_P2.54mm_Vertical"
 			(at 331.47 52.07 0)
 			(hide yes)

Commit message: refining hierarchy
Parts:
- removed C1, C13, C19, C20, C25, C6, C9: 100n, Capacitor_SMD:C_0603_1608Metric_Pad1.08x0.95mm_HandSolder, symbol Device:C
- removed C10, C14: 22p, Capacitor_SMD:C_0603_1608Metric_Pad1.08x0.95mm_HandSolder, symbol Device:C
- removed C11, C16: 1u, Capacitor_SMD:C_0603_1608Metric_Pad1.08x0.95mm_HandSolder, symbol Device:C
- removed C12: 33p, Capacitor_SMD:C_0603_1608Metric_Pad1.08x0.95mm_HandSolder, symbol Device:C
- removed C15, C17, C18: 22u, Capacitor_SMD:C_1210_3225Metric_Pad1.33x2.70mm_HandSolder, symbol Device:C
- removed C2, C4: 4.7u, Capacitor_SMD:C_1206_3216Metric_Pad1.33x1.80mm_HandSolder, symbol Device:C
- removed C21, C22, C23, C7, C8: 1n, Capacitor_SMD:C_0603_1608Metric_Pad1.08x0.95mm_HandSolder, symbol Device:C
- removed C24: 220u, Capacitor_SMD:CP_Elec_10x10, symbol Device:C_Polarized
- removed C26, C27, C3, C5: 10n, Capacitor_SMD:C_0603_1608Metric_Pad1.08x0.95mm_HandSolder, symbol Device:C
- removed D1: BAV99, Package_TO_SOT_SMD:SOT-23, symbol Diode:BAV99
- removed J1: JST B4B XH A, Connector_JST:JST_XH_B4B-XH-A_1x04_P2.50mm_Vertical, symbol Connector:Conn_01x04_Pin
- removed J2: 2.54 mm header, Connector_PinSocket_2.54mm:PinSocket_1x04_P2.54mm_Vertical, symbol Connector:Conn_01x04_Pin
- removed J3: Conn_01x14_Pin, Connector_PinSocket_2.54mm:PinSocket_1x14_P2.54mm_Vertical, symbol Connector:Conn_01x14_Pin
- removed J4: HX JN1.27-2x5 WZ H4.9, Personal:JN1.27-2x5 WZ H4.9, symbol Connector_Generic:Conn_02x05_Odd_Even
- removed J5: USB_C_Receptacle_USB2.0_16P, Personal:USB_C_socket_16P_vertical, symbol Connector:USB_C_Receptacle_USB2.0_16P
- removed J6: Dell DC jack, Personal:Dell DC jack, symbol personal:Dell_DC_barrel_jack
- removed J7: JST B6B XH A, Connector_JST:JST_XH_B6B-XH-A_1x06_P2.50mm_Vertical, symbol Connector:Conn_01x06_Pin
- removed J8: DC barrel assy, Personal:Dell_barrel_assy, symbol personal:DC_barrel_assy
- removed JP1, JP10, JP11, JP12, JP13, JP15, JP16, JP17, JP2, JP21, JP3, JP8: 0R, Personal:Jumper_0603, symbol Device:R
- removed JP14, JP19, JP4, JP5, JP7: 0R, Resistor_SMD:R_1206_3216Metric_Pad1.30x1.75mm_HandSolder, symbol Device:R
- removed JP18, JP22: 0R, Resistor_THT:R_Axial_DIN0204_L3.6mm_D1.6mm_P7.62mm_Horizontal, symbol Device:R
- removed JP20, JP6: 0R, Resistor_SMD:R_0603_1608Metric_Pad0.98x0.95mm_HandSolder, symbol Device:R
- removed JP9: 0R, Resistor_THT:R_Axial_DIN0204_L3.6mm_D1.6mm_P5.08mm_Horizontal, symbol Device:R
- removed L1: 10u, Personal:L_Bourns_SRP6540, symbol Device:L
- removed P1, P12, P13, P15, P16, P2, P22, P25, P27, P28, P30, P31, P32, P33, P43, P44, P45, P47, P6: (no value), symbol personal:Cosmetic_OUT
- removed P10, P11, P14, P17, P18, P19, P20, P21, P23, P24, P26, P29, P3, P37, P38, P39, P4, P40, P41, P42, P5, P7, P8, P9: (no value), symbol personal:Cosmetic_IN
- removed P34, P35, P36, P46, P48, P49: (no value), symbol personal:Cosmetic_IO
- removed R1, R2, R7, R8, R9: 10k, Resistor_SMD:R_0603_1608Metric_Pad0.98x0.95mm_HandSolder, symbol Device:R
- removed R10, R12, R13, R4, R5: 2k2, Resistor_SMD:R_0603_1608Metric_Pad0.98x0.95mm_HandSolder, symbol Device:R
- removed R11: 820, Resistor_SMD:R_0603_1608Metric_Pad0.98x0.95mm_HandSolder, symbol Device:R
- removed R14, R15: 5k1, Resistor_SMD:R_0603_1608Metric_Pad0.98x0.95mm_HandSolder, symbol Device:R
- removed R3: 64.9k, Resistor_SMD:R_0603_1608Metric_Pad0.98x0.95mm_HandSolder, symbol Device:R
- removed R6: 23.2k, Resistor_SMD:R_0603_1608Metric_Pad0.98x0.95mm_HandSolder, symbol Device:R
- removed TFT1: TFT_2.4in_320x240, Personal:Display_240x320_ILI9341_2.4in_no_pads, symbol personal:TFT_2.8_IN_320x240
- removed TP1, TP10, TP11, TP12, TP13, TP14, TP15, TP16, TP17, TP18, TP19, TP2, TP20, TP21, TP3, TP4, TP5, TP6, TP7, TP8, TP9: TestPoint, TestPoint:TestPoint_THTPad_D1.0mm_Drill0.5mm, symbol Connector:TestPoint
- removed U1: LMR380x0, Package_SO:Texas_HSOP-8-1EP_3.9x4.9mm_P1.27mm_ThermalVias, symbol personal:LMR380x0
- removed U2: STM32G431K8Tx, Package_QFP:LQFP-32_7x7mm_P0.8mm, symbol MCU_ST_STM32G4:STM32G431K8Tx
- removed U3: VNH7070, Package_SO:JEITA_SOIC-16_3.9x9.9mm_P1.27mm, symbol personal:VNH7070
- removed U4: USBLC6-2SC6, Package_TO_SOT_SMD:SOT-23-6, symbol Power_Protection:USBLC6-2SC6
- removed Y1: 20 MHz, Crystal:Crystal_SMD_3225-4Pin_3.2x2.5mm_HandSoldering, symbol Device:Crystal_GND24_Small
Connections:
- no-connect marks 9 -> 0
Other:
- added sheet DCDC converter - 3V3 (DCDC_converter_3V3)
- added sheet Limit switch interface (Limit_switch_interface.kicad_sch)
- added sheet Microcontroller (Microcontroller.kicad_sch)
- added sheet Servomotor interface (Servomotor_interface.kicad_sch)
- added sheet Touch TFT (Touch_TFT.kicad_sch)
- note removed: "3.3 V supply"
- note removed: "3D model"
- note removed: "Board mounting"
- note removed: "End of travel switch interface"
- note removed: "Microcontroller"
- note removed: "Motor interface"
- note removed: "SWD header"
- note removed: "TFT display"
- note removed: "USB interface (serial comms port)"

Commit message: append extra sheet
Other:
- removed sheet DCDC converter - 3V3
- added sheet DCDC converter 3V3 (DCDC_converter_3V3.kicad_sch)
Changed lines of the file:
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@@
 			(color 0 0 0 0)
 		)
-		(property "Sheetname" "DCDC converter - 3V3"
+		(property "Sheetname" "DCDC converter 3V3"
 			(at 38.1 62.7884 0)
 			(show_name no)
@@
 			)
 		)
-		(property "Sheetfile" "DCDC_converter_3V3"
+		(property "Sheetfile" "DCDC_converter_3V3.kicad_sch"
 			(at 38.1 89.4846 0)
 			(show_name no)

Commit message: sch2
Other:
- sheet Microcontroller ports: added DISP_CS, DISP_DC, DISP_MISO, DISP_MOSI, DISP_RST, DISP_SCK, TCH_CS, TCH_IRQ; removed none
- sheet Touch TFT ports: added DISP_CS, DISP_DC, DISP_MISO, DISP_MOSI, DISP_RST, DISP_SCK, GND, S3V3, TCH_CS, TCH_IRQ; removed none

Commit message: updated sch template (A4)
Other:
- sheet Touch TFT renamed Display
- sheet Display: file Touch_TFT.kicad_sch -> Display.kicad_sch
- note removed: "${SHEETNAME}"
Changed lines of the file:
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@@
 	(generator_version "10.0")
 	(paper "A4")
-	(text "${SHEETNAME}"
-		(exclude_from_sim no)
-		(at 283.21 14.605 0)
-		(effects
-			(font
-				(face "DejaVu Sans")
-				(size 3.81 3.81)
-				(bold yes)
-				(color 0 0 0 1)
-			)
-			(justify right top)
-		)
-	)
 	(text "Return to front sheet"
 		(exclude_from_sim no)
@@
 				(size 2.032 2.032)
 				(thickness 0.3175)
-				(color 0 0 0 1)
+				(color 0 0 194 1)
 			)
 			(justify left bottom)
@@
 			(color 255 229 191 1)
 		)
-		(property "Sheetname" "Touch TFT"
+		(property "Sheetname" "Display"
 			(at 177.8 100.8884 0)
 			(show_name no)
@@
 			)
 		)
-		(property "Sheetfile" "Touch_TFT.kicad_sch"
+		(property "Sheetfile" "Display.kicad_sch"
 			(at 177.8 140.2846 0)
 			(show_name no)
