File: Touch_TFT.kicad_sch (KiCad schematic)
At the start: 0 parts

Commit message: sch update
Parts:
- added C1: 100n, Capacitor_SMD:C_0603_1608Metric_Pad1.08x0.95mm_HandSolder, symbol Device:C
- added J2: 2.54 mm header, Connector_PinSocket_2.54mm:PinSocket_1x04_P2.54mm_Vertical, symbol Connector:Conn_01x04_Pin
- added J3: Conn_01x14_Pin, Connector_PinSocket_2.54mm:PinSocket_1x14_P2.54mm_Vertical, symbol Connector:Conn_01x14_Pin
- added JP1, JP10, JP11, JP2, JP3, JP8: 0R, Personal:Jumper_0603, symbol Device:R
- added JP4, JP5, JP7: 0R, Resistor_SMD:R_1206_3216Metric_Pad1.30x1.75mm_HandSolder, symbol Device:R
- added JP6: 0R, Resistor_SMD:R_0603_1608Metric_Pad0.98x0.95mm_HandSolder, symbol Device:R
- added JP9: 0R, Resistor_THT:R_Axial_DIN0204_L3.6mm_D1.6mm_P5.08mm_Horizontal, symbol Device:R
- added P1, P2, P6, P78, P83, P84, P85, P86, P87: (no value), symbol personal:Cosmetic_OUT
- added P10, P11, P3, P4, P5, P7, P79, P8, P80, P9: (no value), symbol personal:Cosmetic_IN
- added TFT1: TFT_2.4in_320x240, Personal:Display_240x320_ILI9341_2.4in_no_pads, symbol personal:TFT_2.8_IN_320x240
Connections:
- new net: J3.3 (Pin_3), JP11.2
- new net: J3.10 (Pin_10), JP5.2
- new net: J3.11 (Pin_11), JP4.2
- new net: J3.12 (Pin_12), JP3.2
- new net: J3.13 (Pin_13), JP2.2
- new net: J3.14 (Pin_14), JP1.2
- new net: J3.4 (Pin_4), JP10.2
- new net: J3.5 (Pin_5), JP9.2
- new net: J3.6 (Pin_6), JP8.2
- new net: J3.7 (Pin_7), JP7.2
- new net: J3.9 (Pin_9), JP6.2
- new net DISP_CS: JP11.1, P11.1, P87.1
- new net DISP_DC: JP9.1, P85.1, P9.1
- new net DISP_MISO: JP2.1, JP6.1, P2.1, P6.1, P80.1
- new net DISP_MOSI: JP3.1, JP8.1, P3.1, P8.1, P84.1
- new net DISP_RST: JP10.1, P10.1, P86.1
- new net DISP_SCK: JP5.1, JP7.1, P5.1, P7.1, P83.1
- new net GND: C1.2, J3.2 (Pin_2)
- new net S3V3: C1.1, J3.1 (Pin_1), J3.8 (Pin_8)
- new net TCH_CS: JP4.1, P4.1, P78.1
- new net TCH_IRQ: JP1.1, P1.1, P79.1
- no-connect marks 0 -> 4
Other:
- note added: "3D model"
- note added: "Return to front sheet"

Commit message: reorganised sch and pcb
Other:
- note added: "The display will not be directly soldered to the PCB. Instead, generic 2.54 mm pitch sockets J2 and J3 will be used as connectors."
Changed lines of the file:
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@@
+		)
+	)
+	(text "The display will not\nbe directly soldered\nto the PCB. Instead,\ngeneric 2.54 mm pitch\nsockets J2 and J3 will\nbe used as connectors."
+		(exclude_from_sim no)
+		(at 152.4 73.66 0)
+		(effects
+			(font
+				(size 2.032 2.032)
+				(color 0 0 0 1)
+			)
+			(justify left top)
 		)
 	)
@@
 		(dnp no)
 		(property "Reference" "J2"
-			(at 90.17 82.55 0)
-			(show_name no)
-			(do_not_autoplace no)
+			(at 88.265 83.82 0)
+			(show_name no)
+			(do_not_autoplace no)
