File: Limit_switch_interface.kicad_sch (KiCad schematic)
At the start: 16 parts, among them J1 JST B4B XH A

Commit message: sch update
Other:
- note added: "Return to front sheet"
Changed lines of the file:
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@@
+		)
+	)
+	(text "Return to front sheet"
+		(exclude_from_sim no)
+		(at 12.7 197.485 0)
+		(effects
+			(font
+				(face "DejaVu Sans")
+				(size 2.032 2.032)
+				(thickness 0.3175)
+				(color 0 0 0 1)
+			)
+			(justify left bottom)
+			(href "#1")
 		)
 	)

Commit message: updated sch template (A4)
Other:
- note removed: "${SHEETNAME}"
Changed lines of the file:
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@@
-		)
-	)
-	(text "${SHEETNAME}"
-		(exclude_from_sim no)
-		(at 283.21 14.605 0)
-		(effects
-			(font
-				(face "DejaVu Sans")
-				(size 3.81 3.81)
-				(bold yes)
-				(color 0 0 0 1)
-			)
-			(justify right top)
 		)
 	)
@@
 				(size 2.032 2.032)
 				(thickness 0.3175)
-				(color 0 0 0 1)
+				(color 0 0 194 1)
 			)
 			(justify left bottom)

Commit message: supplier and mpn added
Parts:
- C3, C5: Manufacturer (none) -> Yageo; Manufacturer Part Number (none) -> AC0603KRX7R9BB103
- C7, C8: Manufacturer (none) -> Yageo; Manufacturer Part Number (none) -> AC0603KRX7R9BB102
- J1: value JST B4B XH A -> B4B XH A; Manufacturer (none) -> JST; Manufacturer Part Number (none) -> B4B XH A
- P12, P13, P62, P63: Manufacturer (none) -> NA; Manufacturer Part Number (none) -> NA
- R1, R2: Manufacturer (none) -> YAGEO; Manufacturer Part Number (none) -> AC0603FR-0710KL
- R4, R5: Manufacturer (none) -> YAGEO; Manufacturer Part Number (none) -> AC0603FR-072K2L
- TP19, TP3, TP4: Manufacturer (none) -> NA; Manufacturer Part Number (none) -> NA; now left out of the parts list
