File: Microcontroller.kicad_sch (KiCad schematic)
At the start: 87 parts, among them J2 2.54 mm header, J3 Conn_01x14_Pin, J4 HX JN1.27-2x5 WZ H4.9, J5 USB_C_Receptacle_USB2.0_16P, U2 STM32G431K8Tx, U4 USBLC6-2SC6, Y1 20 MHz

Commit message: sch update
Parts:
- removed C1: 100n, Capacitor_SMD:C_0603_1608Metric_Pad1.08x0.95mm_HandSolder, symbol Device:C
- removed J2: 2.54 mm header, Connector_PinSocket_2.54mm:PinSocket_1x04_P2.54mm_Vertical, symbol Connector:Conn_01x04_Pin
- removed J3: Conn_01x14_Pin, Connector_PinSocket_2.54mm:PinSocket_1x14_P2.54mm_Vertical, symbol Connector:Conn_01x14_Pin
- removed JP1, JP10, JP11, JP2, JP3, JP8: 0R, Personal:Jumper_0603, symbol Device:R
- removed JP4, JP5, JP7: 0R, Resistor_SMD:R_1206_3216Metric_Pad1.30x1.75mm_HandSolder, symbol Device:R
- removed JP6: 0R, Resistor_SMD:R_0603_1608Metric_Pad0.98x0.95mm_HandSolder, symbol Device:R
- removed JP9: 0R, Resistor_THT:R_Axial_DIN0204_L3.6mm_D1.6mm_P5.08mm_Horizontal, symbol Device:R
- removed P1, P2, P6: (no value), symbol personal:Cosmetic_OUT
- removed P10, P11, P3, P4, P5, P7, P8, P9: (no value), symbol personal:Cosmetic_IN
- removed TFT1: TFT_2.4in_320x240, Personal:Display_240x320_ILI9341_2.4in_no_pads, symbol personal:TFT_2.8_IN_320x240
Connections:
- no-connect marks 8 -> 4
Other:
- note added: "Return to front sheet"
- note removed: "3D model"
- note removed: "TFT display"

Commit message: sch2
Parts:
- added P100, P101: (no value), symbol personal:Cosmetic_OUT
- added P94, P95, P96, P97, P98, P99: (no value), symbol personal:Cosmetic_IN
Connections:
- net DISP_CS: now also P96.1
- net DISP_DC: now also P99.1
- net DISP_MISO: now also P100.1
- net DISP_MOSI: now also P98.1
- net DISP_RST: now also P94.1
- net DISP_SCK: now also P97.1
- net TCH_CS: now also P95.1
- net TCH_IRQ: now also P101.1

Commit message: reorganised sch and pcb
Other:
- moved on the sheet: J4, JP14

Commit message: updated sch template (A4)
Other:
- note removed: "${SHEETNAME}"
Changed lines of the file:
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@@
-		)
-	)
-	(text "${SHEETNAME}"
-		(exclude_from_sim no)
-		(at 283.21 14.605 0)
-		(effects
-			(font
-				(face "DejaVu Sans")
-				(size 3.81 3.81)
-				(bold yes)
-				(color 0 0 0 1)
-			)
-			(justify right top)
 		)
 	)
@@
 				(size 2.032 2.032)
 				(thickness 0.3175)
-				(color 0 0 0 1)
+				(color 0 0 194 1)
 			)
 			(justify left bottom)

Commit message: supplier and mpn added
Parts:
- C10, C14: Manufacturer (none) -> Yageo; Manufacturer Part Number (none) -> AC0603JRNPO9BN220
- C11, C16: Manufacturer (none) -> Yageo; Manufacturer Part Number (none) -> AC0603KRX7R7BB105
- C13, C19, C20: Manufacturer (none) -> Yageo; Manufacturer Part Number (none) -> AC0603KRX7R9BB104
- J4: Manufacturer (none) -> HX JN1.27-2x5 WZ H4.9; Manufacturer Part Number (none) -> Hanxia
- J5: Manufacturer (none) -> ChengHaoRan; Manufacturer Part Number (none) -> TFKH5-16L4CC-65
- P100, P101, P14, P15, P16, P17, P18, P19, P20, P21, P22, P23, P24, P25, P26, P27, P28, P29, P30, P31, P32, P33, P34, P35, P36, P37, P38, P46, P47, P48, P49, P53, P58, P59, P60, P61, P64, P65, P66, P67, P94, P95, P96, P97, P98, P99: Manufacturer (none) -> NA; Manufacturer Part Number (none) -> NA
- R14, R15: Manufacturer (none) -> YAGEO; Manufacturer Part Number (none) -> AC0603FR-075K1L
- R8, R9: Manufacturer (none) -> YAGEO; Manufacturer Part Number (none) -> AC0603FR-0710KL
- TP16, TP8, TP9: Manufacturer (none) -> NA; Manufacturer Part Number (none) -> NA; now left out of the parts list
- U2: value STM32G431K8Tx -> STM32G431K8T; Manufacturer (none) -> ST; Manufacturer Part Number (none) -> STM32G431K8T6
- U4: Manufacturer (none) -> ST; Manufacturer Part Number (none) -> USBLC6-2SC6
- Y1: Manufacturer (none) -> KYOCERA AVX; Manufacturer Part Number (none) -> CX3225SB20000H0FLJCC
