File: Servomotor_interface.kicad_sch (KiCad schematic)
At the start: 41 parts, among them J7 JST B6B XH A, U3 VNH7070

Commit message: sch update
Other:
- note added: "Return to front sheet"
Changed lines of the file:
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@@
+		)
+	)
+	(text "Return to front sheet"
+		(exclude_from_sim no)
+		(at 12.7 197.485 0)
+		(effects
+			(font
+				(face "DejaVu Sans")
+				(size 2.032 2.032)
+				(thickness 0.3175)
+				(color 0 0 0 1)
+			)
+			(justify left bottom)
+			(href "#1")
 		)
 	)

Commit message: reorganised sch and pcb
Other:
- moved on the sheet: C21, C22, C23, C24, C25, C26, C27, D1, J7, JP15, JP16, JP17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

Commit message: updated sch template (A4)
Other:
- note removed: "${SHEETNAME}"
Changed lines of the file:
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@@
-		)
-	)
-	(text "${SHEETNAME}"
-		(exclude_from_sim no)
-		(at 283.21 14.605 0)
-		(effects
-			(font
-				(face "DejaVu Sans")
-				(size 3.81 3.81)
-				(bold yes)
-				(color 0 0 0 1)
-			)
-			(justify right top)
 		)
 	)
@@
 				(size 2.032 2.032)
 				(thickness 0.3175)
-				(color 0 0 0 1)
+				(color 0 0 194 1)
 			)
 			(justify left bottom)

Commit message: supplier and mpn added
Parts:
- C21, C22, C23: Manufacturer (none) -> Yageo; Manufacturer Part Number (none) -> AC0603KRX7R9BB102
- C24: Manufacturer (none) -> Panasonic; Manufacturer Part Number (none) -> EEE-FK1H221P
- C25: Manufacturer (none) -> Yageo; Manufacturer Part Number (none) -> AC0603KRX7R9BB104
- C26, C27: Manufacturer (none) -> Yageo; Manufacturer Part Number (none) -> AC0603KRX7R9BB103
- D1: Manufacturer (none) -> Diodes Inc; Manufacturer Part Number (none) -> BAV99Q-7-F
- J7: value JST B6B XH A -> B6B XH A; Manufacturer (none) -> JST; Manufacturer Part Number (none) -> B6B XH A
- P39, P40, P41, P42, P43, P44, P45, P50, P51, P52, P54, P55, P56, P57: Manufacturer (none) -> NA; Manufacturer Part Number (none) -> NA
- R10, R12, R13: Manufacturer (none) -> YAGEO; Manufacturer Part Number (none) -> AC0603FR-072K2L
- R11: Manufacturer (none) -> YAGEO; Manufacturer Part Number (none) -> AC0603FR-07820RL
- TP11, TP12, TP13, TP14, TP15, TP20, TP21: Manufacturer (none) -> NA; Manufacturer Part Number (none) -> NA; now left out of the parts list
- U3: Manufacturer (none) -> ST; Manufacturer Part Number (none) -> VNH7070
